File: MCU_AURA/MCU_AURA.kicad_pcb (KiCad board)
At the start: 4 copper layers, 112 parts, among them J1 TF-CARD_H1.8, J101 USB_C_Receptacle_USB2.0_16P, J2 TC2050-IDC-430, J3 XT30PW-M, J4 532617006, J5 532617004, J500 Screw_Terminal_01x04, J6 532617004, Q300 BSS138, Q301 BSS138, Q302 BSS138, U1 DMN6040SSD-13, U101 SI4825DDY-T1-GE3, U104 AP2127N-1.8, U2 TPS56C230RJER, U200 ESP32-S3-WROOM-1, U201 USBLC6-2SC6, U3 TPS2115ADRBR, U300 ICM-20948, U301 BMP280, U4 TLV62566DBVR

Commit message: Adding Connectors
Parts:
- removed C100, C114, C115: 1u, Capacitor_SMD:C_0402_1005Metric
- removed C101, C102: 22u, Capacitor_SMD:C_1206_3216Metric
- removed C103: 18n, Capacitor_SMD:C_0402_1005Metric
- removed C104, C109, C110, C201, C203, C204, C300, C301, C302, C303, C304, C305: 100n, Capacitor_SMD:C_0402_1005Metric
- removed C105: 100n, Capacitor_SMD:C_0603_1608Metric
- removed C106, C107, C108: 22u, Capacitor_SMD:C_0805_2012Metric
- removed C111, C113, C202: 10u, Capacitor_SMD:C_0402_1005Metric
- removed C112: 4u7, Capacitor_SMD:C_0805_2012Metric
- removed C200: 22u, Capacitor_SMD:C_0402_1005Metric
- removed D1: MMSZ5242B, MMSZ5252B:MMSZ5252B
- removed D100, D102, D103, D104: LED, LED_SMD:LED_0603_1608Metric
- removed H1, H2, H3, H4: MountingHole_Pad, MountingHole:MountingHole_4mm_Pad_Via
- removed J1: TF-CARD_H1.8, TF-CARD_H1_8:TFCARDH18
- removed J101: USB_C_Receptacle_USB2.0_16P, Connector_USB:USB_C_Receptacle_GCT_USB4105-xx-A_16P_TopMnt_Horizontal
- removed J2: TC2050-IDC-430, TC2050-IDC:TC2050-IDC
- removed J3: XT30PW-M, XT30PWM:XT30PWM
- removed J4: 532617006, 532617006:532617006
- removed J5, J6: 532617004, 532617004:532617004
- removed J500: Screw_Terminal_01x04, TerminalBlock_MetzConnect:TerminalBlock_MetzConnect_Type086_RT03404HBLC_1x04_P3.81mm_Horizontal
- removed JP100, JP101: SolderJumper_2_Bridged, Jumper:SolderJumper-2_P1.3mm_Open_RoundedPad1.0x1.5mm
- removed L100: 1u8, CKST0603:CKST0603-1.5uHM
- removed L101: 2u2, Inductor_SMD:L_1008_2520Metric
- removed Q300, Q301, Q302: BSS138, Package_TO_SOT_SMD:SOT-23
- removed R100, R101: 5k1, Resistor_SMD:R_0402_1005Metric
- removed R102: 49k, Resistor_SMD:R_0402_1005Metric
- removed R103: 13k, Resistor_SMD:R_0402_1005Metric
- removed R104: 180k, Resistor_SMD:R_0402_1005Metric
- removed R105: 33k, Resistor_SMD:R_0402_1005Metric
- removed R106: 330k, Resistor_SMD:R_0402_1005Metric
- removed R107: 110k, Resistor_SMD:R_0402_1005Metric
- removed R108: 15k, Resistor_SMD:R_0402_1005Metric
- removed R109, R117: 4k7, Resistor_SMD:R_0402_1005Metric
- removed R110: 100k, Resistor_SMD:R_0402_1005Metric
- removed R111, R115, R500, R503: 220k, Resistor_SMD:R_0402_1005Metric
- removed R112, R501, R504: 22k, Resistor_SMD:R_0402_1005Metric
- removed R113, R120: 1k, Resistor_SMD:R_0402_1005Metric
- removed R116: 680R, Resistor_SMD:R_0402_1005Metric
- removed R118: 540k, Resistor_SMD:R_0402_1005Metric
- removed R119: 120k, Resistor_SMD:R_0402_1005Metric
- removed R200, R205, R206, R300, R301, R302, R502, R505, R506: 10k, Resistor_SMD:R_0402_1005Metric
- removed R201, R202: 27R, Resistor_SMD:R_0402_1005Metric
- removed S1, S2: EVQ-PUC02K, EVQ-PUC02k:EVQPUC02K
- removed TP100, TP101, TP102, TP103, TP104, TP105, TP106, TP107, TP108, TP109, TP110, TP300, TP301, TP302: TestPoint, TestPoint:TestPoint_Pad_D1.0mm
- removed U1: DMN6040SSD-13, DMN6040SSD-13:SOIC127P600X170-8N
- removed U101: SI4825DDY-T1-GE3, SI4825DDY-T1-GE3:SI4825DDY-T1-GE3
- removed U104: AP2127N-1.8, Package_TO_SOT_SMD:SOT-23
- removed U2: TPS56C230RJER, TPS56C230RJER:QFN45P300X300X100-21N-D
- removed U200: ESP32-S3-WROOM-1, RF_Module:ESP32-S3-WROOM-1
- removed U201: USBLC6-2SC6, Package_TO_SOT_SMD:SOT-23-6
- removed U3: TPS2115ADRBR, TPS2115ADRBR:SON65P300X300X100-9N-D
- removed U300: ICM-20948, Sensor_Motion:InvenSense_QFN-24_3x3mm_P0.4mm
- removed U301: BMP280, Package_LGA:Bosch_LGA-8_2x2.5mm_P0.65mm_ClockwisePinNumbering
- removed U4: TLV62566DBVR, TLV62566DBVR:SOT95P280X145-5N

Commit message: Initial Schematic Draft
Parts:
- added C100: 100n, Capacitor_SMD:C_0402_1005Metric, F.Cu at (140.8, 81.0)
- added C101: 100n, Capacitor_SMD:C_0402_1005Metric, F.Cu at (134.2, 80.0)
- added C102: 10u, Capacitor_SMD:C_0402_1005Metric, F.Cu at (134.2, 81.0)
- added C103: 4u7, Capacitor_SMD:C_0805_2012Metric, F.Cu at (141.0, 85.5)
- added C104: 10u, Capacitor_SMD:C_0402_1005Metric, F.Cu at (134.5, 89.0)
- added C105: 1u, Capacitor_SMD:C_0402_1005Metric, F.Cu at (126.0, 88.5)
- added C106: 1u, Capacitor_SMD:C_0402_1005Metric, F.Cu at (126.0, 83.5)
- added C200: 22u, Capacitor_SMD:C_0402_1005Metric, F.Cu at (191.3, 73.2)
- added C201: 100n, Capacitor_SMD:C_0402_1005Metric, F.Cu at (191.3, 75.2)
- added C202: 10u, Capacitor_SMD:C_0402_1005Metric, F.Cu at (191.3, 77.1)
- added C203: 100n, Capacitor_SMD:C_0402_1005Metric, F.Cu at (191.3, 79.1)
- added C204: 100n, Capacitor_SMD:C_0402_1005Metric, F.Cu at (191.3, 81.1)
- added C300: 100n, Capacitor_SMD:C_0402_1005Metric, F.Cu at (224.3, 90.4)
- added C301: 100n, Capacitor_SMD:C_0402_1005Metric, F.Cu at (224.3, 92.4)
- added C302: 100n, Capacitor_SMD:C_0402_1005Metric, F.Cu at (224.3, 94.3)
- added C303: 100n, Capacitor_SMD:C_0402_1005Metric, F.Cu at (112.5, 61.0)
- added C304: 100n, Capacitor_SMD:C_0402_1005Metric, F.Cu at (224.3, 96.3)
- added C305: 100n, Capacitor_SMD:C_0402_1005Metric, F.Cu at (224.3, 98.3)
- added C306: 100n, Capacitor_SMD:C_0402_1005Metric, F.Cu at (224.3, 100.2)
- added D100: LED, LED_SMD:LED_0603_1608Metric, F.Cu at (129.5, 84.5)
- added D103: LED, LED_SMD:LED_0603_1608Metric, F.Cu at (131.6, 84.5)
- added D300: LED, LED_SMD:LED_0603_1608Metric, F.Cu at (209.7, 109.1)
- added H1: MountingHole_Pad, MountingHole:MountingHole_4mm_Pad_Via, F.Cu at (106.0, 94.0)
- added H2: MountingHole_Pad, MountingHole:MountingHole_4mm_Pad_Via, F.Cu at (144.0, 94.0)
- added H3: MountingHole_Pad, MountingHole:MountingHole_4mm_Pad_Via, F.Cu at (106.0, 56.0)
- added H4: MountingHole_Pad, MountingHole:MountingHole_4mm_Pad_Via, F.Cu at (144.0, 56.0)
- added IC1: PCA9685PW,118, PCA9685PW_118:SOP65P640X110-28N, F.Cu at (110.0, 67.0)
- added J1: TF-CARD_H1.8, TF-CARD_H1_8:TFCARDH18, B.Cu at (130.5, 92.0)
- added J100: USB_C_Receptacle_USB2.0_16P, Connector_USB:USB_C_Receptacle_GCT_USB4105-xx-A_16P_TopMnt_Horizontal, F.Cu at (116.0, 96.2)
- added J200: TC2050-IDC-430, TC2050-IDC:TC2050-IDC, F.Cu at (141.8, 66.1)
- added J400: 532617004, 532617004:532617004, F.Cu at (105.1, 84.0)
- added J401: 532617004, 532617004:532617004, B.Cu at (105.1, 84.0)
- added J402: 532617004, 532617004:532617004, B.Cu at (145.2, 66.8)
- added J403: 532617010, 532617010:532617010, F.Cu at (145.2, 75.0)
- added J404: 532617007, 532617007:532617007, B.Cu at (105.1, 69.0)
- added J405: 532617007, 532617007:532617007, B.Cu at (145.2, 81.5)
- added J406: 532617012, 532617012:532617012, B.Cu at (125.0, 55.1)
- added J407: 532614005, 532614005:CONN_532610000-SD_05_MOL, F.Cu at (130.5, 98.0)
- added JP100: SolderJumper_2_Bridged, Jumper:SolderJumper-2_P1.3mm_Open_RoundedPad1.0x1.5mm, F.Cu at (229.2, 57.6)
- added JP101: SolderJumper_2_Bridged, Jumper:SolderJumper-2_P1.3mm_Open_RoundedPad1.0x1.5mm, F.Cu at (229.2, 61.2)
- added L101: 2u2, Inductor_SMD:L_1008_2520Metric, F.Cu at (134.5, 85.5)
- added Q300: BSS138, Package_TO_SOT_SMD:SOT-23, F.Cu at (121.5, 79.7)
- added Q301: BSS138, Package_TO_SOT_SMD:SOT-23, F.Cu at (126.0, 80.0)
- added Q302: BSS138, Package_TO_SOT_SMD:SOT-23, F.Cu at (121.5, 88.7)
- added R100: 5k1, Resistor_SMD:R_0402_1005Metric, F.Cu at (225.6, 41.0)
- added R101: 5k1, Resistor_SMD:R_0402_1005Metric, F.Cu at (225.6, 42.9)
- added R102: 680R, Resistor_SMD:R_0402_1005Metric, F.Cu at (140.8, 79.0)
- added R103: 220k, Resistor_SMD:R_0402_1005Metric, F.Cu at (140.8, 80.0)
- added R104: 4k7, Resistor_SMD:R_0402_1005Metric, F.Cu at (129.6, 87.5)
- added R105: 540k, Resistor_SMD:R_0402_1005Metric, F.Cu at (139.0, 89.0)
- added R106: 120k, Resistor_SMD:R_0402_1005Metric, F.Cu at (140.0, 89.0)
- added R107: 1k, Resistor_SMD:R_0402_1005Metric, F.Cu at (131.5, 87.5)
- added R200: 10k, Resistor_SMD:R_0402_1005Metric, F.Cu at (188.4, 73.2)
- added R201: 27R, Resistor_SMD:R_0402_1005Metric, F.Cu at (188.4, 75.2)
- added R202: 27R, Resistor_SMD:R_0402_1005Metric, F.Cu at (188.4, 77.2)
- added R205: 10k, Resistor_SMD:R_0402_1005Metric, F.Cu at (188.4, 79.2)
- added R206: 10k, Resistor_SMD:R_0402_1005Metric, F.Cu at (188.4, 81.2)
- added R300: 10k, Resistor_SMD:R_0402_1005Metric, F.Cu at (222.4, 106.3)
- added R301: 10k, Resistor_SMD:R_0402_1005Metric, F.Cu at (222.4, 108.3)
- added R302: 10k, Resistor_SMD:R_0402_1005Metric, F.Cu at (118.0, 66.1)
- added R303: 10k, Resistor_SMD:R_0402_1005Metric, F.Cu at (222.4, 110.2)
- added R304: 1k, Resistor_SMD:R_0402_1005Metric, F.Cu at (222.4, 104.3)
- added R400: 10k, Resistor_SMD:R_0402_1005Metric, F.Cu at (105.0, 67.0)
- added R401: 10k, Resistor_SMD:R_0402_1005Metric, F.Cu at (144.5, 86.5)
- added S200: EVQ-PUC02K, EVQ-PUC02k:EVQPUC02K, F.Cu at (102.0, 64.5)
- added S201: EVQ-PUC02K, EVQ-PUC02k:EVQPUC02K, F.Cu at (102.0, 73.5)
- added TP100: TestPoint, TestPoint:TestPoint_Pad_D1.0mm, F.Cu at (228.6, 41.5)
- added TP101: TestPoint, TestPoint:TestPoint_Pad_D1.0mm, F.Cu at (228.6, 44.5)
- added TP102: TestPoint, TestPoint:TestPoint_Pad_D1.0mm, F.Cu at (231.6, 41.5)
- added TP103: TestPoint, TestPoint:TestPoint_Pad_D1.0mm, F.Cu at (231.6, 44.5)
- added TP104: TestPoint, TestPoint:TestPoint_Pad_D1.0mm, F.Cu at (234.7, 41.5)
- added TP105: TestPoint, TestPoint:TestPoint_Pad_D1.0mm, F.Cu at (234.7, 44.5)
- added TP300: TestPoint, TestPoint:TestPoint_Pad_D1.0mm, F.Cu at (219.4, 104.8)
- added TP301: TestPoint, TestPoint:TestPoint_Pad_D1.0mm, F.Cu at (219.4, 107.9)
- added TP302: TestPoint, TestPoint:TestPoint_Pad_D1.0mm, F.Cu at (219.4, 110.9)
- added U100: TPS2115ADRBR, TPS2115ADRBR:SON65P300X300X100-9N-D, F.Cu at (137.5, 80.5)
- added U101: TLV62566DBVR, TLV62566DBVR:SOT95P280X145-5N, F.Cu at (138.0, 85.5)
- added U102: AP2127N-1.8, Package_TO_SOT_SMD:SOT-23, F.Cu at (126.0, 86.0)
- added U200: ESP32-S3-WROOM-1, RF_Module:ESP32-S3-WROOM-1, F.Cu at (125.0, 63.0)
- added U201: USBLC6-2SC6, Package_TO_SOT_SMD:SOT-23-6, F.Cu at (116.0, 89.0)
- added U300: ICM-20948, Sensor_Motion:InvenSense_QFN-24_3x3mm_P0.4mm, F.Cu at (121.5, 84.0)
- added U301: BMP280, Package_LGA:Bosch_LGA-8_2x2.5mm_P0.65mm_ClockwisePinNumbering, F.Cu at (110.0, 84.5)
Other:
- board outline added: 50 x 50 mm

Commit message: Initial draft
Parts:
- JP100, JP101, TP102, TP300, TP301: moved to B.Cu
- moved R100 122.3 mm to (113.5, 90.0), turned to -90 degrees
- moved C305 118.2 mm to (113.0, 58.5), turned to 90 degrees
- moved R101 117.0 mm to (118.5, 90.0), turned to -90 degrees
- moved TP104 112.9 mm to (133.0, 90.5)
- moved R304 112.3 mm to (111.5, 87.0), turned to 180 degrees
- moved TP105 110.2 mm to (132.0, 84.5)
- moved TP103 104.7 mm to (137.5, 90.5)
- moved D300 103.3 mm to (108.7, 87.0), turned to 180 degrees
- moved C301 103.1 mm to (121.5, 84.0), turned to 180 degrees
- moved R300 102.7 mm to (122.5, 82.5), turned to 180 degrees
- moved TP102 102.5 mm to (137.5, 82.0), turned to 180 degrees
- moved TP101 102.0 mm to (134.5, 84.0)
- moved C300 101.8 mm to (122.5, 88.5), turned to 180 degrees
- moved R301 99.3 mm to (126.5, 82.5), turned to 180 degrees
- moved C302 98.0 mm to (126.5, 88.5)
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Other:
- outline, holes or cut-outs redrawn

Commit message: Started Routing
Parts:
- added C100: 10u, Capacitor_SMD:C_0402_1005Metric, F.Cu at (123.8, 94.9)
- added C101: 1u, Capacitor_SMD:C_0402_1005Metric, F.Cu at (124.8, 94.9)
- added C102: 100n, Capacitor_SMD:C_0402_1005Metric, F.Cu at (125.8, 94.9)
- added C400: 10u, Capacitor_SMD:C_0402_1005Metric, F.Cu at (136.0, 78.8)
- added C401: 1u, Capacitor_SMD:C_0402_1005Metric, F.Cu at (136.0, 77.7)
- added C402: 100n, Capacitor_SMD:C_0402_1005Metric, F.Cu at (136.0, 76.8)
- added D100: TPD1E05U06DPYR, TPD1E05U06DPYR:DIO_TPD1E05U06DPYR, F.Cu at (119.3, 91.3)
- added D101: TPD1E05U06DPYR, TPD1E05U06DPYR:DIO_TPD1E05U06DPYR, F.Cu at (114.7, 91.3)
- added D102: TPD1E05U06DPYR, TPD1E05U06DPYR:DIO_TPD1E05U06DPYR, F.Cu at (122.7, 94.9)
- added D400: TPD1E05U06DPYR, TPD1E05U06DPYR:DIO_TPD1E05U06DPYR, F.Cu at (141.4, 77.0)
- added D401: TPD1E05U06DPYR, TPD1E05U06DPYR:DIO_TPD1E05U06DPYR, F.Cu at (144.4, 71.8)
- added D402: TPD1E05U06DPYR, TPD1E05U06DPYR:DIO_TPD1E05U06DPYR, F.Cu at (144.4, 73.1)
- added D403: TPD1E05U06DPYR, TPD1E05U06DPYR:DIO_TPD1E05U06DPYR, F.Cu at (144.4, 74.4)
- added D404: TPD1E05U06DPYR, TPD1E05U06DPYR:DIO_TPD1E05U06DPYR, F.Cu at (142.6, 84.3)
- added D405: TPD1E05U06DPYR, TPD1E05U06DPYR:DIO_TPD1E05U06DPYR, F.Cu at (142.6, 83.0)
- added D406: TPD1E05U06DPYR, TPD1E05U06DPYR:DIO_TPD1E05U06DPYR, F.Cu at (142.6, 81.7)
- added D407: TPD1E05U06DPYR, TPD1E05U06DPYR:DIO_TPD1E05U06DPYR, F.Cu at (143.1, 67.7)
- added D408: TPD1E05U06DPYR, TPD1E05U06DPYR:DIO_TPD1E05U06DPYR, F.Cu at (143.1, 66.5)
- added D409: TPD1E05U06DPYR, TPD1E05U06DPYR:DIO_TPD1E05U06DPYR, F.Cu at (107.0, 83.2)
- added D410: TPD1E05U06DPYR, TPD1E05U06DPYR:DIO_TPD1E05U06DPYR, F.Cu at (107.0, 84.8)
- added J408: 532617004, 532610471:53261-0471, B.Cu at (136.0, 54.3)
- added JP200: SolderJumper_2_Bridged, Jumper:SolderJumper-2_P1.3mm_Open_RoundedPad1.0x1.5mm, B.Cu at (122.0, 84.4)
- added R1: 22R, Resistor_SMD:R_0402_1005Metric, F.Cu at (129.8, 84.8)
- added R105: 10k, Resistor_SMD:R_0402_1005Metric, B.Cu at (143.8, 86.8)
- added R109: 10k, Resistor_SMD:R_0402_1005Metric, B.Cu at (138.8, 89.8)
- added R2: 22R, Resistor_SMD:R_0402_1005Metric, F.Cu at (135.8, 66.6)
- added TP105: TestPoint, TestPoint:TestPoint_Pad_D1.0mm, B.Cu at (136.9, 91.2)
- H1, H2, H3, H4: footprint MountingHole:MountingHole_4mm_Pad_Via -> MountingHole:MountingHole_3.2mm_M3_Pad_Via
- J400, J401: footprint 532617004:532617004 -> 532610471:53261-0471
- J402: footprint 532617004:532617004 -> 532610471:53261-0471; moved to F.Cu
- J403: value 532617010 -> 532617012; footprint 532617010:532617010 -> 532611271:53261-1271; moved to B.Cu
- J404: footprint 532617007:532617007 -> 532610771:532610771
- J405: footprint 532617007:532617007 -> 532610771:532610771; moved to F.Cu
- J406: footprint 532617012:532617012 -> 532611271:53261-1271
- J407: value 532614005 -> 532617007; footprint 532614005:CONN_532610000-SD_05_MOL -> 532610771:532610771
- R102: value 680R -> 270R
- R103: value 220k -> 10k
- R106: renamed from R105; value 540k -> 68k
- R107: renamed from R106; value 120k -> 15k
- R201, R202: value 27R -> 22R
- TP103, TP302: moved to B.Cu
- TP106: renamed from TP105; moved to B.Cu
- moved J404 39.8 mm to (133.0, 97.4), turned to 0 degrees
- moved TP104 37.1 mm to (111.9, 60.0)
- moved R401 37.0 mm to (114.2, 65.2)
- moved J1 33.1 mm to (107.5, 68.2), turned to 90 degrees
- moved U301 30.5 mm to (109.5, 81.4), turned to 180 degrees
- moved C201 28.5 mm to (114.2, 59.0), turned to 180 degrees
- moved C306 28.0 mm to (114.2, 69.2), turned to 180 degrees
- moved R300 27.7 mm to (137.2, 59.0), turned to 0 degrees
- moved R301 27.5 mm to (140.8, 59.0), turned to 0 degrees
- moved C301 26.1 mm to (141.6, 67.2), turned to 90 degrees
- moved Q301 24.7 mm to (140.8, 61.8), turned to -90 degrees
- moved TP300 24.1 mm to (137.2, 60.8)
- moved C300 24.0 mm to (137.5, 69.8), turned to -90 degrees
- moved U300 23.7 mm to (139.0, 66.8)
- moved C108 23.6 mm to (141.2, 69.8), turned to 90 degrees
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- renumbered C100 to C103, C101 to C104, C102 to C105, C103 to C106, C104 to C107, C105 to C108, C106 to C109, D100 to D103, D103 to D104, R107 to R108
Connections:
- net /100_Power/ILIM_5V_SW renamed /100_Power/ILIM_5V
- net Net-(IC1-~{OE}) renamed /300_Digital_Peripherals/MUX_OE
- C203 pad 1: /200_ESP32/RST -> /200_ESP32/EN
- C204 pad 1: /200_ESP32/EN -> /200_ESP32/RST
- J200 pad 1: +3V3 -> /200_ESP32/JTAG_3V3
- J403 pad 1: +5V -> GND
- J403 pad 10: GND -> +5V
- J403 pad 11: (no net) -> +5V
- J403 pad 12: (no net) -> +5V
- J403 pad 2: +5V -> GND
- J403 pad 3: +3V3 -> GND
- J403 pad 4: SCL -> +3V3
- J403 pad 6: GND -> SCL
- J403 pad 7: MSFT_1 -> GND
- J403 pad 8: MSFT_2 -> MSFT_1
- J403 pad 9: GND -> MSFT_2
- J407 pad 2: GPS_TX -> +3V3
- J407 pad 3: GPS_RX -> GPS_TX
- J407 pad 4: GPS_INT -> GPS_RX
- J407 pad 5: GND -> GPS_INT
- J407 pad 6: (no net) -> GND
- J407 pad 7: (no net) -> GND
- R100 pad 2: /100_Power/CC1 -> /100_Power/CC2
- R101 pad 2: /100_Power/CC2 -> /100_Power/CC1
- S200 pad 2: /200_ESP32/RST -> GND
- S200 pad 3: GND -> /200_ESP32/EN
- S201 pad 2: /200_ESP32/EN -> GND
- S201 pad 3: GND -> /200_ESP32/RST
- U101 pad 1: +5V_FILT -> /100_Power/PG_3V3
- U200 pad 32: /200_ESP32/TCK -> /200_ESP32/TCK_D
- U200 pad 33: /200_ESP32/TDO -> /200_ESP32/TDO_D
- U200 pad 38: unconnected-(U200-IO2-Pad38) -> ICM_INT
- U200 pad 39: unconnected-(U200-IO1-Pad39) -> RC_RX
- U200 pad 8: ICM_INT -> unconnected-(U200-IO15-Pad8)
Routing:
- net SDA: track 0.00 -> 94.3 mm, vias 0 -> 6
- net SCL: track 0.00 -> 90.7 mm, vias 0 -> 6
- net EXT_CS: track 0.00 -> 52.9 mm, vias 0 -> 2
- net EXT_RST: track 0.00 -> 52.0 mm, vias 0 -> 2
- net MISO: track 0.00 -> 45.0 mm, vias 0 -> 3
- net MOSI: track 0.00 -> 44.9 mm, vias 0 -> 3
- net SCK: track 0.00 -> 43.9 mm, vias 0 -> 3
- net +1V8: track 0.00 -> 41.2 mm, vias 0 -> 3
- net /200_ESP32/RST: track 0.00 -> 38.8 mm, vias 0 -> 2
- net +3V3: track 0.00 -> 32.1 mm, vias 0 -> 22
- net LED: track 0.00 -> 31.8 mm, vias 0 -> 2
- net /200_ESP32/TDO: track 0.00 -> 31.7 mm, vias 0 -> 2
- net +5V_FILT: track 0.00 -> 31.3 mm, vias 0 -> 7
- net +VUSB: track 0.00 -> 29.6 mm, vias 0 -> 13
- net RF_CS: track 0.00 -> 29.6 mm, vias 0 -> 1
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- added copper zone on F.Cu, net +3V3
- added copper zone on In1.Cu, net +3V3
- added copper zone on In2.Cu, net +3V3
- added copper zone on B.Cu, net +5V
- added copper zone on F.Cu, net +5V
- added copper zone on B.Cu, net +5V_FILT
- added copper zone on F.Cu, net +5V_FILT
- added copper zone on B.Cu, net +VUSB
- added copper zone on F.Cu, net +VUSB
- added copper zone on F.Cu, net /100_Power/SW_3V3
- added copper zone on B.Cu, net GND
- added copper zone on F.Cu, net GND
- added copper zone on In1.Cu, net GND
Other:
- board text added: "1V8"
- board text added: "3V3"
- board text added: "5V"
- board text added: "FB"
- board text added: "GPS"
- board text added: "I2C"
- board text added: "INT"
- board text added: "JTAG"
- board text added: "PG"
- board text added: "POWER"
- board text added: "RADIO"
- board text added: "SCL"
- board text added: "SD"
- board text added: "SDA"
- board text added: "SERVOS"
- board text added: "SPI"
- board text added: "STAT"
- board text added: "UART"
- board text added: "USB"
- board text added: "VUSB"

Commit message: First fully routed version
Parts:
- added R302: 10k, Resistor_SMD:R_0402_1005Metric, F.Cu at (135.8, 69.2)
- added R303: 10k, Resistor_SMD:R_0402_1005Metric, F.Cu at (137.2, 75.5)
- C306: moved to B.Cu
- moved R401 26.0 mm to (133.0, 83.2), turned to 90 degrees
- moved TP104 14.5 mm to (109.0, 74.2)
- moved C305 3.36 mm to (112.0, 82.1), turned to 0 degrees
- moved C306 3.25 mm to (117.5, 69.2), turned to 0 degrees
- moved C304 3.12 mm to (112.0, 80.8)
- moved R105 2.75 mm to (143.8, 84.0)
- moved C302 0.48 mm to (139.2, 70.2)
- moved C108 0.45 mm to (140.8, 69.8)
- moved U301 0.30 mm to (109.5, 81.1), turned to 90 degrees
- moved C300 0.25 mm to (137.2, 69.8)
- renumbered R302 to R304, R304 to R305, R303 to R306
Connections:
- H1 pad 1: unconnected-(H1-Pad1)_5 -> GND
- H2 pad 1: unconnected-(H2-Pad1)_1 -> GND
- H3 pad 1: unconnected-(H3-Pad1)_2 -> GND
- H4 pad 1: unconnected-(H4-Pad1)_4 -> GND
- U200 pad 31: unconnected-(U200-IO38-Pad31) -> ICM_INT
- U200 pad 38: ICM_INT -> unconnected-(U200-IO2-Pad38)
Routing:
- net GPS_RX: track 1.60 -> 80.4 mm, vias 0 -> 4
- net GPS_TX: track 1.55 -> 78.0 mm, vias 0 -> 4
- net GND: track 14.1 -> 78.7 mm, vias 9 -> 67
- net MSFT_2: track 0.00 -> 54.1 mm, vias 0 -> 3
- net MSFT_1: track 0.00 -> 52.7 mm, vias 0 -> 3
- net GPS_INT: track 1.55 -> 50.1 mm, vias 0 -> 6
- net /200_ESP32/EN: track 18.4 -> 38.1 mm
- net +3V3: track 32.1 -> 47.1 mm, vias 22 -> 34
- net ICM_INT: track 15.1 -> 5.47 mm
- net MOSI: track 44.9 -> 53.9 mm, vias 3 -> 4
- net +5V_FILT: track 31.3 -> 37.4 mm
- net MISO: track 45.0 -> 50.8 mm, vias 3 -> 4
- net +1V8: track 41.2 -> 46.5 mm, vias 3 -> 4
- net +VUSB: track 29.6 -> 33.6 mm, vias 13 -> 14
- net SCL: track 90.7 -> 94.3 mm
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
Commit message: First version
Parts:
- J100: footprint Connector_USB:USB_C_Receptacle_GCT_USB4105-xx-A_16P_TopMnt_Horizontal -> USB-C:USB_C_Receptacle_GCT_USB4105-xx-A_16P_TopMnt_Horizontal
- moved C102 15.9 mm to (110.0, 96.3), turned to 180 degrees
- moved C101 14.8 mm to (110.0, 95.3), turned to 180 degrees
- moved C100 13.8 mm to (110.0, 94.3), turned to 180 degrees
- moved D102 12.8 mm to (110.0, 93.2), turned to 180 degrees
- moved TP100 5.09 mm to (129.7, 90.0)
- moved D100 1.84 mm to (119.3, 89.5)
- moved D101 1.84 mm to (114.7, 89.5)
- moved J100 1.84 mm to (117.0, 95.8)
- moved R100 1.84 mm to (120.5, 89.4)
- moved R101 1.84 mm to (113.5, 89.5)
- moved U201 1.84 mm to (117.0, 88.9)
Routing:
- net RF_RST: track 27.6 -> 33.6 mm, vias 1 -> 3
- net RF_CS: track 29.6 -> 35.2 mm, vias 1 -> 3
- net GND: track 78.7 -> 74.9 mm, vias 67 -> 66
- net GPS_RX: track 80.4 -> 77.7 mm
- net GPS_TX: track 78.0 -> 75.5 mm
- net +5V_FILT: track 37.4 -> 38.6 mm
- net /200_ESP32/USB_MCU_D-: track 21.8 -> 21.2 mm
- net /200_ESP32/USB_MCU_D+: track 21.8 -> 21.1 mm
- net +VUSB: track 33.6 -> 33.8 mm, vias 14 -> 15

Commit message: Second Iteration
Parts:
- moved R401 5.42 mm to (133.2, 77.8)
- moved D104 0.10 mm to (109.3, 86.1)
- moved R108 0.10 mm to (112.0, 86.1)
Connections:
- J100 pad S1: unconnected-(J100-SHIELD-PadS1) -> (no net)
Routing:
- net EXT_CS: track 55.2 -> 53.2 mm
- net GND: track 74.9 -> 76.5 mm, vias 66 -> 67
- net SCK: track 46.4 -> 45.9 mm
- net MISO: track 50.8 -> 50.3 mm
- net +3V3: track 47.1 -> 47.6 mm, vias 34 -> 35
- net unconnected-(J200-Pad10): vias 1 -> 0
- removed copper zone on In1.Cu, net +3V3
