File: MCU_AURA/Power.kicad_sch (KiCad schematic)
At the start: 43 parts, among them J100 USB_C_Receptacle_USB2.0_16P, U100 TPS2115ADRBR, U101 TLV62566DBVR, U102 AP2127N-1.8

Commit message: Production Files for MCU
Parts:
- R104: value 4k7 -> 1k
- R106: value 68k -> 6k8
- R107: value 15k -> 1k5
- R108: value 1k -> 470R

Commit message: CPL file finalised for MCU
Parts:
- C106: footprint Capacitor_SMD:C_0805_2012Metric -> Capacitor_SMD:C_0402_1005Metric
Changed lines of the file:
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@@
 			)
 		)
-		(property "Footprint" "Capacitor_SMD:C_0805_2012Metric"
+		(property "Footprint" "Capacitor_SMD:C_0402_1005Metric"
 			(at 47.9552 121.92 0)
 			(effects
