File: FPGA_AURA/Power_Regulation.kicad_sch (KiCad schematic)
At the start: 52 parts, among them U200 ADP5014, U4 TPS51200DRCR

Commit message: Continuing the FTDI
Changed lines of the file:
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@@
-		)
-	)
-	(bus_entry
-		(at 158.75 154.94)
-		(size 2.54 2.54)
-		(stroke
-			(width 0)
-			(type default)
 		)
 	)
